File: SolarMPPT.sch (EAGLE design)
At the start: 36 parts, among them J2 1X2-3.5MM, J3 1X2-3.5MM, J6 1X2-3.5MM, U3 LTC1155, U7 LM22674MRX-5.0

Commit message: added mounting holes, art, and generally cleaned up before ordering!
Parts:
- added C4, C5: (no value), rcl:C-US050-024X044
Connections:
- net +18V: now also C4.1
- net GND: now also C4.2, C5.2
- net N$10: now also C5.1
Other:
- note removed: "reroute to pairs?"
Changed lines of the file:
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@@
 <part name="GND2" library="supply1" library_urn="urn:adsk.eagle:library:371" deviceset="GND" device=""/>
 <part name="JP1" library="pinhead" library_urn="urn:adsk.eagle:library:325" deviceset="PINHD-1X13" device="" package3d_urn="urn:adsk.eagle:package:22421/2"/>
+<part name="C4" library="rcl" library_urn="urn:adsk.eagle:library:334" deviceset="C-US" device="050-024X044" package3d_urn="urn:adsk.eagle:package:23643/1"/>
+<part name="C5" library="rcl" library_urn="urn:adsk.eagle:library:334" deviceset="C-US" device="050-024X044" package3d_urn="urn:adsk.eagle:package:23643/1"/>
 </parts>
 <sheets>
@@
 <text x="-71.12" y="281.94" size="1.778" layer="97" rot="MR0">NC</text>
 <text x="-152.4" y="256.54" size="1.778" layer="91">Add fuses</text>
-<text x="-152.4" y="233.68" size="1.778" layer="91">reroute to pairs?</text>
 <text x="25.4" y="218.44" size="7.62" layer="91">add uart</text>
 <text x="-73.66" y="119.38" size="1.778" layer="91">EPD breakout</text>
@@
 <attribute name="NAME" x="-84.455" y="92.71" size="1.778" layer="95" rot="MR270"/>
 <attribute name="VALUE" x="-45.72" y="92.71" size="1.778" layer="96" rot="MR270"/>
+</instance>
+<instance part="C4" gate="G$1" x="-58.42" y="185.42" smashed="yes">
+<attribute name="NAME" x="-57.404" y="186.055" size="1.778" layer="95"/>
+<attribute name="VALUE" x="-57.404" y="181.229" size="1.778" layer="96"/>
+</instance>
+<instance part="C5" gate="G$1" x="-81.28" y="157.48" smashed="yes">
+<attribute name="NAME" x="-80.264" y="158.115" size="1.778" layer="95"/>
+<attribute name="VALUE" x="-80.264" y="153.289" size="1.778" layer="96"/>
 </instance>
 </instances>
@@
 <wire x1="-73.66" y1="160.02" x2="-73.66" y2="152.4" width="0.1524" layer="91"/>
 <wire x1="-73.66" y1="160.02" x2="-60.96" y2="160.02" width="0.1524" layer="91"/>
+<pinref part="C5" gate="G$1" pin="2"/>
+<wire x1="-81.28" y1="152.4" x2="-73.66" y2="152.4" width="0.1524" layer="91"/>
+<junction x="-73.66" y="152.4"/>
 </segment>
 <segment>
@@
 <pinref part="GND19" gate="1" pin="GND"/>
 <wire x1="-68.58" y1="180.34" x2="-81.28" y2="180.34" width="0.1524" layer="91"/>
+<pinref part="C4" gate="G$1" pin="2"/>
+<wire x1="-58.42" y1="180.34" x2="-68.58" y2="180.34" width="0.1524" layer="91"/>
+<junction x="-68.58" y="180.34"/>
 </segment>
 <segment>
@@
 <wire x1="-81.28" y1="187.96" x2="-68.58" y2="187.96" width="0.1524" layer="91"/>
 <junction x="-81.28" y="187.96"/>
+<pinref part="C4" gate="G$1" pin="1"/>
+<wire x1="-58.42" y1="187.96" x2="-68.58" y2="187.96" width="0.1524" layer="91"/>
+<junction x="-68.58" y="187.96"/>
 </segment>
 <segment>
@@
 <pinref part="BIGBOB" gate="G$1" pin="2"/>
 <pinref part="COUT1" gate="G$1" pin="1"/>
-<wire x1="-86.36" y1="167.64" x2="-73.66" y2="167.64" width="0.1524" layer="91"/>
+<wire x1="-86.36" y1="167.64" x2="-81.28" y2="167.64" width="0.1524" layer="91"/>
 <pinref part="COUT2" gate="G$1" pin="1"/>
+<wire x1="-81.28" y1="167.64" x2="-73.66" y2="167.64" width="0.1524" layer="91"/>
 <wire x1="-73.66" y1="167.64" x2="-60.96" y2="167.64" width="0.1524" layer="91"/>
 <junction x="-73.66" y="167.64"/>
@@
 <junction x="-60.96" y="167.64"/>
 <junction x="-45.72" y="167.64"/>
-</segment>
-</net>
+<pinref part="C5" gate="G$1" pin="1"/>
+<wire x1="-81.28" y1="160.02" x2="-81.28" y2="167.64" width="0.1524" layer="91"/>
+<junction x="-81.28" y="167.64"/>
+</segment>
+</net>

Commit message: Went back and forth with osh getting it right, this version was ORDERED
Changed lines of the file:
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@@
 <wire x1="-127" y1="152.4" x2="-127" y2="147.32" width="0.1524" layer="91"/>
 <wire x1="-127" y1="147.32" x2="-127" y2="139.7" width="0.1524" layer="91"/>
+<pinref part="DNP" gate="G$1" pin="A"/>
 <wire x1="-127" y1="147.32" x2="-114.3" y2="147.32" width="0.1524" layer="91"/>
-<pinref part="DNP" gate="G$1" pin="A"/>
 <wire x1="-114.3" y1="147.32" x2="-114.3" y2="152.4" width="0.1524" layer="91"/>
+<junction x="-127" y="147.32"/>
 </segment>
 <segment>
@@
 <pinref part="GND21" gate="1" pin="GND"/>
 <pinref part="COUT2" gate="G$1" pin="2"/>
-<wire x1="-73.66" y1="160.02" x2="-73.66" y2="152.4" width="0.1524" layer="91"/>
 <wire x1="-73.66" y1="160.02" x2="-60.96" y2="160.02" width="0.1524" layer="91"/>
 <pinref part="C5" gate="G$1" pin="2"/>
 <wire x1="-81.28" y1="152.4" x2="-73.66" y2="152.4" width="0.1524" layer="91"/>
 <junction x="-73.66" y="152.4"/>
+<wire x1="-73.66" y1="160.02" x2="-73.66" y2="152.4" width="0.1524" layer="91"/>
+<junction x="-73.66" y="160.02"/>
 </segment>
 <segment>

Commit message: Created digikey cart, updated schematic with components
Parts:
- C1: value 1uF 50v -> 10uF 50v
- C2: value 4.7uF 50v -> 10uF 50v
- C4, C5: value (none) -> big radial cap
- CCFIL1, CVDD4: value 4.7uF -> 10uF
- CCUR1: value 1uF -> 10uF
- CVDD3: value 100nF -> 10nF
- DNP: value MBR0520LT3G -> PMEG6010CEH
Changed lines of the file:
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@@
 </classes>
 <parts>
-<part name="CVDD3" library="rcl" library_urn="urn:adsk.eagle:library:334" deviceset="C-US" device="C0805" package3d_urn="urn:adsk.eagle:package:23617/2" value="100nF"/>
-<part name="CVDD4" library="rcl" library_urn="urn:adsk.eagle:library:334" deviceset="C-US" device="C0805" package3d_urn="urn:adsk.eagle:package:23617/2" value="4.7uF"/>
+<part name="CVDD3" library="rcl" library_urn="urn:adsk.eagle:library:334" deviceset="C-US" device="C0805" package3d_urn="urn:adsk.eagle:package:23617/2" value="10nF"/>
+<part name="CVDD4" library="rcl" library_urn="urn:adsk.eagle:library:334" deviceset="C-US" device="C0805" package3d_urn="urn:adsk.eagle:package:23617/2" value="10uF"/>
 <part name="+3V10" library="supply1" library_urn="urn:adsk.eagle:library:371" deviceset="+3V3" device=""/>
 <part name="GND8" library="supply1" library_urn="urn:adsk.eagle:library:371" deviceset="GND" device=""/>
@@
 <part name="RCFIL1" library="rcl" library_urn="urn:adsk.eagle:library:334" deviceset="R-US_" device="R0805" package3d_urn="urn:adsk.eagle:package:23553/2"/>
 <part name="RCFIL2" library="rcl" library_urn="urn:adsk.eagle:library:334" deviceset="R-US_" device="R0805" package3d_urn="urn:adsk.eagle:package:23553/2"/>
-<part name="CCFIL1" library="rcl" library_urn="urn:adsk.eagle:library:334" deviceset="C-US" device="C0805" package3d_urn="urn:adsk.eagle:package:23617/2" value="4.7uF"/>
+<part name="CCFIL1" library="rcl" library_urn="urn:adsk.eagle:library:334" deviceset="C-US" device="C0805" package3d_urn="urn:adsk.eagle:package:23617/2" value="10uF"/>
 <part name="U2" library="FormE" deviceset="INA225" device="VSSOP"/>
 <part name="+3V11" library="supply1" library_urn="urn:adsk.eagle:library:371" deviceset="+3V3" device=""/>
@@
 <part name="GND19" library="supply1" library_urn="urn:adsk.eagle:library:371" deviceset="GND" device=""/>
 <part name="GND21" library="supply1" library_urn="urn:adsk.eagle:library:371" deviceset="GND" device=""/>
-<part name="DNP" library="FormE" deviceset="MBR0520LT3G" device="" value="MBR0520LT3G"/>
-<part name="CCUR1" library="rcl" library_urn="urn:adsk.eagle:library:334" deviceset="C-US" device="C0805" package3d_urn="urn:adsk.eagle:package:23617/2" value="1uF"/>
+<part name="DNP" library="FormE" deviceset="MBR0520LT3G" device="" value="PMEG6010CEH"/>
+<part name="CCUR1" library="rcl" library_urn="urn:adsk.eagle:library:334" deviceset="C-US" device="C0805" package3d_urn="urn:adsk.eagle:package:23617/2" value="10uF"/>
 <part name="P+9" library="supply1" deviceset="+5V" device=""/>
 <part name="U7" library="FormE" deviceset="LM22674" device="" value="LM22674MRX-5.0">
@@
 </part>
 <part name="GND27" library="supply1" deviceset="GND" device=""/>
-<part name="C1" library="rcl" deviceset="C-US" device="C0805" value="1uF 50v">
+<part name="C1" library="rcl" deviceset="C-US" device="C0805" value="10uF 50v">
 <attribute name="PARTNO" value="UMK212BJ105KG-T"/>
 </part>
-<part name="C2" library="rcl" deviceset="C-US" device="C1206" value="4.7uF 50v">
+<part name="C2" library="rcl" deviceset="C-US" device="C1206" value="10uF 50v">
 <attribute name="PARTNO" value="GRM31CR71H475KA12L"/>
 </part>
@@
 <part name="GND2" library="supply1" library_urn="urn:adsk.eagle:library:371" deviceset="GND" device=""/>
 <part name="JP1" library="pinhead" library_urn="urn:adsk.eagle:library:325" deviceset="PINHD-1X13" device="" package3d_urn="urn:adsk.eagle:package:22421/2"/>
-<part name="C4" library="rcl" library_urn="urn:adsk.eagle:library:334" deviceset="C-US" device="050-024X044" package3d_urn="urn:adsk.eagle:package:23643/1"/>
-<part name="C5" library="rcl" library_urn="urn:adsk.eagle:library:334" deviceset="C-US" device="050-024X044" package3d_urn="urn:adsk.eagle:package:23643/1"/>
+<part name="C4" library="rcl" library_urn="urn:adsk.eagle:library:334" deviceset="C-US" device="050-024X044" package3d_urn="urn:adsk.eagle:package:23643/1" value="big radial cap"/>
+<part name="C5" library="rcl" library_urn="urn:adsk.eagle:library:334" deviceset="C-US" device="050-024X044" package3d_urn="urn:adsk.eagle:package:23643/1" value="big radial cap"/>
 </parts>
 <sheets>
